File: neighbor-template.kicad_pcb (KiCad board)
At the start: 4 copper layers, 70.7 x 53.3 mm, 7 parts, among them J1 NEIGHBOR1, J2 NEIGHBOR2, J7 BONUS_ROW

Commit message: remove copyright and license from schematic so they are not imposed upon projects that copy this template update dates in schematic and layout
Other:
- board text added: "22 September 2019"
- board text removed: "27 September 2015"
Changed lines of the file:
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@@
   (gr_line (start 177.9016 92.3544) (end 177.8508 94.0054) (angle 90) (layer Edge.Cuts) (width 0.15))
   (gr_line (start 177.9524 90.5002) (end 177.9016 92.3544) (angle 90) (layer Edge.Cuts) (width 0.15))
-  (gr_text "27 September 2015" (at 153.4414 114.4016) (layer F.SilkS)
+  (gr_text "22 September 2019" (at 153.4414 114.4016) (layer F.SilkS)
     (effects (font (size 1.016 0.762) (thickness 0.1524)))
   )

Commit message: copy gsg-kicad-lib footprints to local library remove gsg-kicad-lib dependency
Parts:
- J1, J2: footprint gsg-modules:HEADER-2x20 -> neighbor:HEADER-2x20
- J7: footprint gsg-modules:HEADER-1x20 -> neighbor:HEADER-1x20
- MH1, MH2, MH3, MH4: footprint gsg-modules:HOLE126MIL-COPPER -> neighbor:HOLE126MIL-COPPER
Changed lines of the file:
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@@
     (add_net VCC)
   )
-  (module gsg-modules:HEADER-1x20 (layer F.Cu)
+  (module neighbor:HEADER-1x20 (layer F.Cu)
     (at 146.05 76.2)
     (tags CONN)
@@
       (net 2 VCC))
   )
-  (module gsg-modules:HEADER-2x20 (layer F.Cu)
+  (module neighbor:HEADER-2x20 (layer F.Cu)
     (at 146.05 118.11)
     (tags CONN)
@@
       (die_length 0.08382))
   )
-  (module gsg-modules:HEADER-2x20 (layer F.Cu)
+  (module neighbor:HEADER-2x20 (layer F.Cu)
     (at 146.05 72.39)
     (tags CONN)
@@
       (die_length 0.08382))
   )
-  (module gsg-modules:HOLE126MIL-COPPER (layer F.Cu)
+  (module neighbor:HOLE126MIL-COPPER (layer F.Cu)
     (at 115.57 74.93)
     (fp_text reference MH1 (at 0 0) (layer F.SilkS) hide
@@
       (net 1 GND))
   )
-  (module gsg-modules:HOLE126MIL-COPPER (layer F.Cu)
+  (module neighbor:HOLE126MIL-COPPER (layer F.Cu)
     (at 115.57 115.57)
     (fp_text reference MH2 (at 0 0) (layer F.SilkS) hide
@@
       (net 1 GND))
   )
-  (module gsg-modules:HOLE126MIL-COPPER (layer F.Cu)
+  (module neighbor:HOLE126MIL-COPPER (layer F.Cu)
     (at 176.53 118.11)
     (fp_text reference MH3 (at 0 0) (layer F.SilkS) hide
@@
       (net 1 GND))
   )
-  (module gsg-modules:HOLE126MIL-COPPER (layer F.Cu)
+  (module neighbor:HOLE126MIL-COPPER (layer F.Cu)
     (at 176.53 72.39)
     (fp_text reference MH4 (at 0 0) (layer F.SilkS) hide
